Commit message: gazebo works, rviz does not

File: urdf/robot.xacro (robot description, xacro)
@@ -66,5 +66,5 @@
   </xacro:macro>
 <!-- Dummy link and joint-->
-  <link name="dummy">
+<!-- <link name="dummy">
   </link>
   <joint name="dummy_to_body" type="fixed">
@@ -72,9 +72,8 @@
     <child link="body"/>
     <parent link="dummy"/>
-  </joint>
+  </joint> -->
 <!-- Body Configuration -->
   <link name="body">
     <!-- pose and inertial -->
-    <pose>0 0 0.1 0 0 0</pose>
     <inertial>
       <mass value="5"/>
