Commit message: working urdf and xacro

File: urdf/my_robot.urdf (robot description, URDF)
Before this commit: robot m2wr, 11 links, 10 joints
Links:
- link arm_link_01: geometry collision cylinder length=0.5 radius=0.04; visual cylinder length=0.5 radius=0.04
- link arm_link_02: geometry collision cylinder length=0.5 radius=0.04; visual cylinder length=0.5 radius=0.04
- link arm_link_03: geometry collision cylinder length=0.3 radius=0.04; visual cylinder length=0.08 radius=0.04
Joints:
- joint arm_joint_01: origin xyz=0 0 0.09 rpy=0 0 0 -> xyz=0 0 0.16 rpy=0 0 0
- joint arm_joint_02: origin xyz=0 0 0.04 rpy=0 0 0 -> xyz=0 0 0.21 rpy=0 0 0
- joint arm_joint_03: origin xyz=0 0 0.08 rpy=0 0 0 -> xyz=0 0 0.3 rpy=0 0 0

File: urdf/my_robot.xacro (robot description, xacro)
@@ -147,5 +147,5 @@
   	  <origin xyz="0 0 0" rpy="0 0 0"/>
       <geometry>
-        <cylinder radius="0.04" length="0.08"/>
+        <cylinder radius="0.04" length="0.5"/>
       </geometry>
   	</collision>
@@ -153,5 +153,5 @@
   	  <origin xyz="0 0 0" rpy="0 0 0"/>
       <geometry>
-        <cylinder radius="0.04" length="0.08"/>
+        <cylinder radius="0.04" length="0.5"/>
       </geometry>
       <material name="red" />
@@ -161,5 +161,5 @@
   	<axis xyz="0 0 1"/>
   	<limit effort="1000.0" lower="-3.14" upper="3.14" velocity="0.2"/>
-  	<origin rpy="0 0 0" xyz="0 0 0.09"/>
+  	<origin rpy="0 0 0" xyz="0 0 0.16"/>
   	<parent link="arm_base_link"/>
   	<child link="arm_link_01"/>
@@ -172,13 +172,13 @@
   	</inertial>
   	<collision>
-  	  <origin xyz="0 0 0.04" rpy="0 0 0"/>
-      <geometry>
-        <cylinder radius="0.04" length="0.08"/>
-      </geometry>
-  	</collision>
-  	<visual>
-  	  <origin xyz="0 0 0.04" rpy="0 0 0"/>
-      <geometry>
-        <cylinder radius="0.04" length="0.08"/>
+  	  <origin xyz="0 0 0.16" rpy="0 0 0"/>
+      <geometry>
+        <cylinder radius="0.04" length="0.5"/>
+      </geometry>
+  	</collision>
+  	<visual>
+  	  <origin xyz="0 0 0.16" rpy="0 0 0"/>
+      <geometry>
+        <cylinder radius="0.04" length="0.5"/>
       </geometry>
       <material name="red" />
@@ -188,5 +188,5 @@
   	<axis xyz="1 0 0"/>
   	<limit effort="1000.0" lower="-1.8" upper="1.8" velocity="0.2"/>
-  	<origin rpy="0 0 0" xyz="0 0 0.04"/>
+  	<origin rpy="0 0 0" xyz="0 0 0.21"/>
   	<parent link="arm_link_01"/>
   	<child link="arm_link_02"/>
@@ -201,12 +201,12 @@
   	  <origin xyz="0 0 0.04" rpy="0 0 0"/>
       <geometry>
+        <cylinder radius="0.04" length="0.3"/>
+      </geometry>
+  	</collision>
+  	<visual>
+  	  <origin xyz="0 0 0.04" rpy="0 0 0"/>
+      <geometry>
         <cylinder radius="0.04" length="0.08"/>
       </geometry>
-  	</collision>
-  	<visual>
-  	  <origin xyz="0 0 0.04" rpy="0 0 0"/>
-      <geometry>
-        <cylinder radius="0.04" length="0.08"/>
-      </geometry>
       <material name="red" />
   	</visual>
@@ -215,5 +215,5 @@
   	<axis xyz="1 0 0"/>
   	<limit effort="1000.0" lower="-1.8" upper="1.8" velocity="0.2"/>
-  	<origin rpy="0 0 0" xyz="0 0 0.08"/>
+  	<origin rpy="0 0 0" xyz="0 0 0.3"/>
   	<parent link="arm_link_02"/>
   	<child link="arm_link_03"/>

Commit message: works, needs commenting

File: urdf/my_robot.urdf (robot description, URDF)
Before this commit: robot m2wr, 11 links, 10 joints
Joints:
- joint joint_left_wheel: origin xyz=-0.05 -0.15 0 rpy=0 0 0 -> xyz=-0.05 0.15 0 rpy=0 0 0
- joint joint_right_wheel: origin xyz=-0.05 0.15 0 rpy=0 0 0 -> xyz=-0.05 -0.15 0 rpy=0 0 0

Commit message: works, needs commenting

File: urdf/my_robot.urdf (robot description, URDF)
Before this commit: robot m2wr, 11 links, 10 joints
Links:
- link arm_base_link: geometry collision box size=0.1 0.1 0.1; visual box size=0.1 0.1 0.4
Joints:
- joint arm_base_to_base: origin xyz=0 0 0.085 rpy=0 0 0 -> xyz=0 0 0.275 rpy=0 0 0
- joint arm_joint_01: origin xyz=0 0 0.16 rpy=0 0 0 -> xyz=0 0 0.36 rpy=0 0 0
